File: pcb/trompbot-1.sch (KiCad schematic (older format))
At the start: 17 parts, among them K11 RELAY, K12 RELAY, P1 CONN_3, P2 CONN_3, P3 CONN_2, P4 CONN_2, P5 CONN_4, P6 CONN_3, P7 CONN_2, P8 CONN_2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

Commit message: fixed let footprint (soldermask bottom), added farnell order codes to components and made BOM
Parts:
- C1: order code (none) -> 2112751
- D1: order code (none) -> 1779664
- K11, K12: order code (none) -> 1081622
- P1, P2, P6: order code (none) -> 1798944
- P3, P4, P7, P8: order code (none) -> 1798941
- P5: order code (none) -> 1798945
- P9: ordercode (none) -> 1835265
- R3: value 470R -> 150R; ordercode (none) -> 1700226
- R4: value 10R -> 150R; ordercode (none) -> 1700226
- U1: order code (none) -> 1853793
- U2: order code (none) -> 1869471
Changed lines of the file:
@@
-EESchema Schematic File Version 2  date Tue 19 Jun 2012 11:34:25 PM CEST
+EESchema Schematic File Version 2  date Wed 18 Jul 2012 12:37:47 AM CEST
 LIBS:power
 LIBS:ti-launchpad
@@
 encoding utf-8
 Sheet 1 1
-Title ""
-Date "19 jun 2012"
-Rev ""
-Comp ""
-Comment1 ""
+Title "KekBot breakout board - kekbot.org"
+Date "17 jul 2012"
+Rev "2"
+Comp "(c) 2012 KekkeTek - www.kekketek.nl"
+Comment1 "CC-BY-SA -see: creativecommons.org"
 Comment2 ""
 Comment3 ""
@@
 P 3550 3350
 F 0 "R4" V 3630 3350 50  0000 C CNN
-F 1 "10R" V 3550 3350 50  0000 C CNN
+F 1 "150R" V 3550 3350 50  0000 C CNN
+F 4 "1700226" H 3550 3350 60  0001 C CNN "ordercode"
 	1    3550 3350
 	1    0    0    1
@@
 F 0 "C1" H 3600 3900 50  0000 L CNN
 F 1 "0.1uF" H 3600 3700 50  0000 L CNN
+F 4 "2112751" H 3550 3800 60  0001 C CNN "order code"
 	1    3550 3800
 	-1   0    0    -1
@@
 F 0 "U2" H 2000 3900 60  0000 C CNN
 F 1 "SFH-5110" H 2000 3800 60  0000 C CNN
+F 4 "1869471" H 2000 3700 60  0001 C CNN "order code"
 	1    2000 3700
 	0    -1   -1   0
@@
 P 3900 3350
 F 0 "R3" V 3980 3350 50  0000 C CNN
-F 1 "470R" V 3900 3350 50  0000 C CNN
+F 1 "150R" V 3900 3350 50  0000 C CNN
+F 4 "1700226" H 3900 3350 60  0001 C CNN "ordercode"
 	1    3900 3350
 	-1   0    0    1
@@
 F 0 "D1" H 3900 3900 50  0000 C CNN
 F 1 "LED" H 3900 3700 50  0000 C CNN
+F 4 "1779664" H 3900 3800 60  0001 C CNN "order code"
 	1    3900 3800
 	0    -1   1    0
@@
 F 0 "P1" V 9800 4600 50  0000 C CNN
 F 1 "CONN_3" V 9900 4600 40  0000 C CNN
+F 4 "1798944 " H 9850 4600 60  0001 C CNN "order code"
 	1    9850 4600
 	1    0    0    -1
@@
 F 0 "P2" V 3400 4800 50  0000 C CNN
 F 1 "CONN_3" V 3500 4800 40  0000 C CNN
+F 4 "1798944 " H 3450 4800 60  0001 C CNN "order code"
 	1    3450 4800
 	-1   0    0    -1
@@
 F 0 "K11" H 8950 6550 60  0000 C CNN
 F 1 "RELAY" H 8850 6650 60  0000 C CNN
+F 4 "1081622" H 8850 6350 60  0001 C CNN "order code"
 	1    8850 6350
 	1    0    0    -1
@@
 F 0 "P3" V 9800 5600 40  0000 C CNN
 F 1 "CONN_2" V 9900 5600 40  0000 C CNN
+F 4 "1798941" H 9850 5600 60  0001 C CNN "order code"
 	1    9850 5600
 	1    0    0    -1
@@
 F 0 "P4" V 9800 6350 40  0000 C CNN
 F 1 "CONN_2" V 9900 6350 40  0000 C CNN
+F 4 "1798941" H 9850 6350 60  0001 C CNN "order code"
 	1    9850 6350
 	1    0    0    -1
@@
 F 0 "K12" H 8950 5800 60  0000 C CNN
 F 1 "RELAY" H 8850 5900 60  0000 C CNN
+F 4 "1081622" H 8850 5600 60  0001 C CNN "order code"
 	1    8850 5600
 	1    0    0    -1
@@
 F 0 "P5" V 9800 4000 50  0000 C CNN
 F 1 "CONN_4" V 9900 4000 50  0000 C CNN
+F 4 "1798945" H 9850 4000 60  0001 C CNN "order code"
 	1    9850 4000
 	1    0    0    -1
@@
 F 0 "P6" V 2650 2900 50  0000 C CNN
 F 1 "CONN_3" V 2750 2900 40  0000 C CNN
+F 4 "1798944 " H 2700 2900 60  0001 C CNN "order code"
 	1    2700 2900
 	-1   0    0    -1
@@
 F 0 "U1" H 6400 4750 60  0000 C CNN
 F 1 "TI-LAUNCHPAD" H 6350 4850 60  0000 C CNN
+F 4 "1853793" H 6400 4250 60  0001 C CNN "order code"
 	1    6400 4250
 	1    0    0    -1
@@
 F 0 "P7" V 2050 4600 40  0000 C CNN
 F 1 "CONN_2" V 2150 4600 40  0000 C CNN
+F 4 "1798941" H 2100 4600 60  0001 C CNN "order code"
 	1    2100 4600
 	-1   0    0    -1
@@
 F 0 "P8" V 3750 2450 40  0000 C CNN
 F 1 "CONN_2" V 3850 2450 40  0000 C CNN
+F 4 "1798941" H 3800 2450 60  0001 C CNN "order code"
 	1    3800 2450
 	-1   0    0    -1
@@
 F 0 "P9" H 4330 4200 40  0000 L CNN
 F 1 "CONN_1" H 4250 4255 30  0001 C CNN
+F 4 "1835265 " H 4250 4200 60  0001 C CNN "ordercode"
 	1    4250 4200
 	-1   0    0    1
